File: _autosave-carteV1.kicad_pcb (KiCad board)
At the start: 2 copper layers, 0 parts

Commit message: Insertion capa pour découplage + new footprint
Parts:
- added BARRETTE_8V: VAL**, BARRETTE_8V, F.Cu at (0.00, 0.00)
Changed lines of the file:
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@@
-(kicad_pcb (version 3) (host pcbnew "(2014-01-10 BZR 4027)-stable")
+(kicad_pcb (version 3) (host pcbnew "(2013-07-07 BZR 4022)-stable")
   (general
     (links 0)
@@
     (tracks 0)
     (zones 0)
-    (modules 0)
+    (modules 1)
     (nets 1)
   )
   (page A3)
   (layers
-    (15 F.Cu signal)
-    (0 B.Cu signal)
-    (16 B.Adhes user)
-    (17 F.Adhes user)
-    (18 B.Paste user)
-    (19 F.Paste user)
-    (20 B.SilkS user)
-    (21 F.SilkS user)
-    (22 B.Mask user)
-    (23 F.Mask user)
-    (24 Dwgs.User user)
+    (15 Dessus.Cu signal)
+    (0 Dessous.Cu signal)
+    (16 Dessous.Adhes user)
+    (17 Dessus.Adhes user)
+    (18 Dessous.Pate user)
+    (19 Dessus.Pate user)
+    (20 Dessous.SilkS user)
+    (21 Dessus.SilkS user)
+    (22 Dessous.Masque user)
+    (23 Dessus.Masque user)
+    (24 Dessin.User user)
     (25 Cmts.User user)
     (26 Eco1.User user)
     (27 Eco2.User user)
-    (28 Edge.Cuts user)
+    (28 Contours.Ci user)
   )
   (setup
@@
   )
   (net 0 "")
-  (net_class Default "This is the default net class."
+  (net_class Default "Ceci est la Netclass par défaut"
     (clearance 0.254)
     (trace_width 0.254)
@@
     (add_net "")
   )
+  (module BARRETTE_8V (layer Dessus.Cu)
+    (at 0 0)
+    (fp_text reference BARRETTE_8V (at 0 -3.81) (layer Dessus.SilkS)
+      (effects (font (size 1 1) (thickness 0.15)))
+    )
+    (fp_text value VAL** (at 0 -2.54) (layer Dessus.SilkS) hide
+      (effects (font (size 1 1) (thickness 0.15)))
+    )
+    (fp_line (start -10.035 -1.27) (end -10.035 1.27) (layer Dessus.SilkS) (width 0.15))
+    (fp_line (start 10.035 -1.27) (end 10.035 1.27) (layer Dessus.SilkS) (width 0.15))
+    (fp_line (start 10.035 -1.27) (end -10.035 -1.27) (layer Dessus.SilkS) (width 0.15))
+    (fp_line (start -10.035 1.27) (end 10.035 1.27) (layer Dessus.SilkS) (width 0.15))
+    (pad 1 thru_hole circle (at -8.89 0) (size 2 2) (drill 1.02)
+      (layers *.Mask Dessous.Cu Dessous.SilkS)
+    )
+    (pad 2 thru_hole circle (at -6.35 0) (size 2 2) (drill 1.02)
+      (layers *.Mask Dessous.Cu Dessus.SilkS)
+    )
+    (pad 3 thru_hole circle (at -3.81 0) (size 2 2) (drill 1.02)
+      (layers *.Mask Dessous.Cu Dessus.SilkS)
+    )
+    (pad 4 thru_hole circle (at -1.27 0) (size 2 2) (drill 1.02)
+      (layers *.Mask Dessous.Cu Dessus.SilkS)
+    )
+    (pad 5 thru_hole circle (at 1.27 0) (size 2 2) (drill 1.02)
+      (layers *.Mask Dessous.Cu Dessus.SilkS)
+    )
+    (pad 6 thru_hole circle (at 3.81 0) (size 2 2) (drill 1.02)
+      (layers *.Mask Dessous.Cu Dessus.SilkS)
+    )
+    (pad 7 thru_hole circle (at 6.35 0) (size 2 2) (drill 1.02)
+      (layers *.Mask Dessous.Cu Dessus.SilkS)
+    )
+    (pad 8 thru_hole circle (at 8.89 0) (size 2 2) (drill 1.02)
+      (layers *.Mask Dessous.Cu Dessus.SilkS)
+    )
+  )
 )
